Commit message: Progress

File: roboticstoolbox/models/xacro/franka_description/robots/panda_arm.xacro (robot description, xacro)
@@ -267,5 +267,5 @@
         <origin xyz="0 0 0.08" rpy="0 0 0"/>
         <geometry>
-          <sphere radius="${0.04+safety_distance}"  />
+          <sphere radius="${0.025+safety_distance}"  />
         </geometry>
       </collision>
