Commit message: stderr fix

File: roboticstoolbox/models/xacro/franka_description/robots/hand.xacro (robot description, xacro)
@@ -62,5 +62,4 @@
     <link name="${ns}_rightfinger">
       <visual>
-        <origin xyz="0 0 0" rpy="0 0 ${pi}"/>
         <geometry>
           <mesh filename="package://franka_description/meshes/visual/finger.dae"/>

Commit message: fixed panda model

File: roboticstoolbox/models/xacro/franka_description/robots/hand.xacro (robot description, xacro)
@@ -62,4 +62,5 @@
     <link name="${ns}_rightfinger">
       <visual>
+        <origin xyz="0 0 0" rpy="0 0 ${pi}"/>
         <geometry>
           <mesh filename="package://franka_description/meshes/visual/finger.dae"/>
