Commit message: model fixed

File: roboticstoolbox/models/URDF/xacro/franka_description/robots/frankie_arm.xacro (robot description, xacro)
@@ -12,15 +12,4 @@
     </xacro:unless>
     <link name="${arm_id}_base0">
-      <visual>
-        <origin xyz="0 0 0.15" rpy="0 0 0"/>
-        <geometry>
-          <box size="0.6 0.4 0.3" />
-        </geometry>
-      </visual>
-      <collision>
-        <geometry>
-          <box size="0.4 0.6 0.5" />
-        </geometry>
-      </collision>
     </link>
     <link name="${arm_id}_base1">
@@ -42,4 +31,16 @@
     <link name="${arm_id}_link0">
       <visual>
+        <origin xyz="0 0 -0.15" rpy="0 0 0"/>
+        <geometry>
+          <box size="0.6 0.4 0.3" />
+        </geometry>
+      </visual>
+      <collision>
+        <origin xyz="0 0 -0.15" rpy="0 0 0"/>
+        <geometry>
+          <box size="0.6 0.4 0.3" />
+        </geometry>
+      </collision>
+      <visual>
         <geometry>
           <mesh filename="package://${description_pkg}/meshes/visual/link0.dae"/>
