Commit message: fknm

File: rtb-data/rtbdata/xacro/kuka_description/kuka_lbr_iiwa/urdf/lbr_iiwa_14_r820_macro.xacro (robot description, xacro)
@@ -1,5 +1,5 @@
 <?xml version="1.0"?>
 <robot xmlns:xacro="http://wiki.ros.org/xacro">
-  <xacro:macro name="kuka_lbr_iiwa_14_r820" params="prefix">
+  <xacro:macro name="kuka_lbr_iiwa_14_r820" params="prefix description_pkg:='kuka_description/kuka_lbr_iiwa'">
     <!-- link list -->
     <link name="${prefix}base_link">
@@ -7,5 +7,5 @@
         <origin xyz="0 0 0" rpy="0 0 0" />
         <geometry>
-          <mesh filename="package://kuka_lbr_iiwa_support/meshes/lbr_iiwa_14_r820/visual/base_link.dae" />
+          <mesh filename="package://${description_pkg}/meshes/lbr_iiwa_14_r820/visual/base_link.dae" />
         </geometry>
       </visual>
@@ -13,5 +13,5 @@
         <origin xyz="0 0 0" rpy="0 0 0" />
         <geometry>
-          <mesh filename="package://kuka_lbr_iiwa_support/meshes/lbr_iiwa_14_r820/collision/base_link.stl" />
+          <mesh filename="package://${description_pkg}/meshes/lbr_iiwa_14_r820/collision/base_link.stl" />
         </geometry>
       </collision>
@@ -21,5 +21,5 @@
         <origin xyz="0 0 0" rpy="0 0 0" />
         <geometry>
-          <mesh filename="package://kuka_lbr_iiwa_support/meshes/lbr_iiwa_14_r820/visual/link_1.dae" />
+          <mesh filename="package://${description_pkg}/meshes/lbr_iiwa_14_r820/visual/link_1.dae" />
         </geometry>
       </visual>
@@ -27,5 +27,5 @@
         <origin xyz="0 0 0" rpy="0 0 0" />
         <geometry>
-          <mesh filename="package://kuka_lbr_iiwa_support/meshes/lbr_iiwa_14_r820/collision/link_1.stl" />
+          <mesh filename="package://${description_pkg}/meshes/lbr_iiwa_14_r820/collision/link_1.stl" />
         </geometry>
       </collision>
@@ -35,5 +35,5 @@
         <origin xyz="0 0 0" rpy="0 0 0" />
         <geometry>
-          <mesh filename="package://kuka_lbr_iiwa_support/meshes/lbr_iiwa_14_r820/visual/link_2.dae" />
+          <mesh filename="package://${description_pkg}/meshes/lbr_iiwa_14_r820/visual/link_2.dae" />
         </geometry>
       </visual>
@@ -41,5 +41,5 @@
         <origin xyz="0 0 0" rpy="0 0 0" />
         <geometry>
-          <mesh filename="package://kuka_lbr_iiwa_support/meshes/lbr_iiwa_14_r820/collision/link_2.stl" />
+          <mesh filename="package://${description_pkg}/meshes/lbr_iiwa_14_r820/collision/link_2.stl" />
         </geometry>
       </collision>
@@ -49,5 +49,5 @@
         <origin xyz="0 0 0" rpy="0 0 0" />
         <geometry>
-          <mesh filename="package://kuka_lbr_iiwa_support/meshes/lbr_iiwa_14_r820/visual/link_3.dae" />
+          <mesh filename="package://${description_pkg}/meshes/lbr_iiwa_14_r820/visual/link_3.dae" />
         </geometry>
       </visual>
@@ -55,5 +55,5 @@
         <origin xyz="0 0 0" rpy="0 0 0" />
         <geometry>
-          <mesh filename="package://kuka_lbr_iiwa_support/meshes/lbr_iiwa_14_r820/collision/link_3.stl" />
+          <mesh filename="package://${description_pkg}/meshes/lbr_iiwa_14_r820/collision/link_3.stl" />
         </geometry>
       </collision>
@@ -63,5 +63,5 @@
         <origin xyz="0 0 0" rpy="0 0 0" />
         <geometry>
-          <mesh filename="package://kuka_lbr_iiwa_support/meshes/lbr_iiwa_14_r820/visual/link_4.dae" />
+          <mesh filename="package://${description_pkg}/meshes/lbr_iiwa_14_r820/visual/link_4.dae" />
         </geometry>
       </visual>
@@ -69,5 +69,5 @@
         <origin xyz="0 0 0" rpy="0 0 0" />
         <geometry>
-          <mesh filename="package://kuka_lbr_iiwa_support/meshes/lbr_iiwa_14_r820/collision/link_4.stl" />
+          <mesh filename="package://${description_pkg}/meshes/lbr_iiwa_14_r820/collision/link_4.stl" />
         </geometry>
       </collision>
@@ -77,5 +77,5 @@
         <origin xyz="0 0 0" rpy="0 0 0" />
         <geometry>
-          <mesh filename="package://kuka_lbr_iiwa_support/meshes/lbr_iiwa_14_r820/visual/link_5.dae" />
+          <mesh filename="package://${description_pkg}/meshes/lbr_iiwa_14_r820/visual/link_5.dae" />
         </geometry>
       </visual>
@@ -83,5 +83,5 @@
         <origin xyz="0 0 0" rpy="0 0 0" />
         <geometry>
-          <mesh filename="package://kuka_lbr_iiwa_support/meshes/lbr_iiwa_14_r820/collision/link_5.stl" />
+          <mesh filename="package://${description_pkg}/meshes/lbr_iiwa_14_r820/collision/link_5.stl" />
         </geometry>
       </collision>
@@ -91,5 +91,5 @@
         <origin xyz="0 0 0" rpy="0 0 0" />
         <geometry>
-          <mesh filename="package://kuka_lbr_iiwa_support/meshes/lbr_iiwa_14_r820/visual/link_6.dae" />
+          <mesh filename="package://${description_pkg}/meshes/lbr_iiwa_14_r820/visual/link_6.dae" />
         </geometry>
       </visual>
@@ -97,5 +97,5 @@
         <origin xyz="0 0 0" rpy="0 0 0" />
         <geometry>
-          <mesh filename="package://kuka_lbr_iiwa_support/meshes/lbr_iiwa_14_r820/collision/link_6.stl" />
+          <mesh filename="package://${description_pkg}/meshes/lbr_iiwa_14_r820/collision/link_6.stl" />
         </geometry>
       </collision>
@@ -105,5 +105,5 @@
         <origin xyz="0 0 0" rpy="0 0 0" />
         <geometry>
-          <mesh filename="package://kuka_lbr_iiwa_support/meshes/lbr_iiwa_14_r820/visual/link_7.dae" />
+          <mesh filename="package://${description_pkg}/meshes/lbr_iiwa_14_r820/visual/link_7.dae" />
         </geometry>
       </visual>
@@ -111,5 +111,5 @@
         <origin xyz="0 0 0" rpy="0 0 0" />
         <geometry>
-          <mesh filename="package://kuka_lbr_iiwa_support/meshes/lbr_iiwa_14_r820/collision/link_7.stl" />
+          <mesh filename="package://${description_pkg}/meshes/lbr_iiwa_14_r820/collision/link_7.stl" />
         </geometry>
       </collision>
