Commit message: Omron model

File: rtb-data/rtbdata/xacro/franka_description/robots/frankie_arm.xacro (robot description, xacro)
@@ -23,5 +23,5 @@
     </joint>
     <joint name="${arm_id}_base_joint2" type="prismatic">
-      <origin rpy="0 0 0" xyz="0 0 0.3"/>
+      <origin rpy="0 0 0" xyz="0 0 0.38"/>
       <parent link="${arm_id}_base1"/>
       <child link="${arm_id}_link0"/>
@@ -31,13 +31,15 @@
     <link name="${arm_id}_link0">
       <visual>
-        <origin xyz="0 0 -0.15" rpy="0 0 0"/>
-        <geometry>
-          <box size="0.6 0.4 0.3" />
-        </geometry>
-      </visual>
-      <collision>
-        <origin xyz="0 0 -0.15" rpy="0 0 0"/>
-        <geometry>
-          <box size="0.6 0.4 0.3" />
+        <!-- <origin xyz="0 0 -0.15" rpy="0 0 0"/> -->
+        <origin xyz="0 0 -0.38" rpy="0 0 0"/>
+        <geometry>
+          <!-- <box size="0.6 0.4 0.3" /> -->
+          <mesh filename="package://${description_pkg}/meshes/visual/omron.dae"/>
+        </geometry>
+      </visual>
+      <collision>
+        <origin xyz="0 0 -0.19" rpy="0 0 0"/>
+        <geometry>
+          <box size="0.68 0.47 0.38" />
         </geometry>
       </collision>

Commit message: removed homogenous points

File: rtb-data/rtbdata/xacro/franka_description/robots/frankie_arm.xacro (robot description, xacro)
@@ -45,9 +45,10 @@
       </collision>
       <visual>
+        <origin xyz="0.15 0 0" rpy="0 0 0"/>
         <geometry>
           <mesh filename="package://${description_pkg}/meshes/visual/link0.dae"/>
         </geometry>
       </visual>
-      <collision>
+      <!-- <collision>
         <origin xyz="-0.075 0 0.06" rpy="0 ${pi/2} 0"/>
         <geometry>
@@ -66,5 +67,5 @@
           <sphere radius="${0.06+safety_distance}" />
         </geometry>
-      </collision>
+      </collision> -->
     </link>
     <link name="${arm_id}_link1">
@@ -95,5 +96,5 @@
     <joint name="${arm_id}_joint1" type="revolute">
       <safety_controller k_position="100.0" k_velocity="40.0" soft_lower_limit="-2.8973" soft_upper_limit="2.8973"/>
-      <origin rpy="0 0 0" xyz="0 0 0.333"/>
+      <origin rpy="0 0 0" xyz="0.15 0 0.333"/>
       <parent link="${arm_id}_link0"/>
       <child link="${arm_id}_link1"/>
