Commit message: wip: rework xacro and URDF parsing
- replace xacro preprocessor with xacrodoc
- move all Robot/Link logic out of tools/urdf/urdf.py into robot/RobotURDF
- rework models/URDF classes for new structure

TODO:
- lots of commented out code
- ugly solution to avoiding circular imports, fix up __init__ files
- tests NOT PASSING

File: rtb-data/rtbdata/xacro/trossen_descriptions/urdf/vx300.urdf.xacro (robot description, xacro)
@@ -9,8 +9,8 @@
   <xacro:property name="urdf_loc" value="$(arg external_urdf_loc)"/>
   <xacro:if value="$(arg load_gazebo_configs)">
-    <xacro:include filename="$(find interbotix_gazebo)/config/interbotix_texture.gazebo"/>
+    <xacro:include filename="$(find trossen_gazebo)/config/trossen_texture.gazebo"/>
   </xacro:if>
-  <material name="interbotix_black">
-    <texture filename="package://interbotix_descriptions/meshes/interbotix_black.png"/>
+  <material name="trossen_black">
+    <texture filename="package://trossen_descriptions/meshes/trossen_black.png"/>
   </material>
   <xacro:if value="$(arg use_world_frame)">
@@ -25,12 +25,12 @@
       <origin rpy="0 0 ${pi/2}" xyz="0 0 0"/>
       <geometry>
-        <mesh filename="package://interbotix_descriptions/meshes/meshes_vx300/VXA-300-M-1-Base.stl" scale="0.001 0.001 0.001"/>
-      </geometry>
-      <material name="interbotix_black"/>
-    </visual>
-    <collision>
-      <origin rpy="0 0 ${pi/2}" xyz="0 0 0"/>
-      <geometry>
-        <mesh filename="package://interbotix_descriptions/meshes/meshes_vx300/VXA-300-M-1-Base.stl" scale="0.001 0.001 0.001"/>
+        <mesh filename="package://trossen_descriptions/meshes/meshes_vx300/VXA-300-M-1-Base.stl" scale="0.001 0.001 0.001"/>
+      </geometry>
+      <material name="trossen_black"/>
+    </visual>
+    <collision>
+      <origin rpy="0 0 ${pi/2}" xyz="0 0 0"/>
+      <geometry>
+        <mesh filename="package://trossen_descriptions/meshes/meshes_vx300/VXA-300-M-1-Base.stl" scale="0.001 0.001 0.001"/>
       </geometry>
     </collision>
@@ -61,12 +61,12 @@
       <origin rpy="0 0 ${pi/2}" xyz="0 0 -0.003"/>
       <geometry>
-        <mesh filename="package://interbotix_descriptions/meshes/meshes_vx300/VXA-300-M-2-Shoulder.stl" scale="0.001 0.001 0.001"/>
-      </geometry>
-      <material name="interbotix_black"/>
+        <mesh filename="package://trossen_descriptions/meshes/meshes_vx300/VXA-300-M-2-Shoulder.stl" scale="0.001 0.001 0.001"/>
+      </geometry>
+      <material name="trossen_black"/>
     </visual>
     <collision>
       <origin rpy="0 0 ${pi/2}" xyz="0 0 -0.003"/>
       <geometry>
-        <mesh filename="package://interbotix_descriptions/meshes/meshes_vx300/VXA-300-M-2-Shoulder.stl" scale="0.001 0.001 0.001"/>
+        <mesh filename="package://trossen_descriptions/meshes/meshes_vx300/VXA-300-M-2-Shoulder.stl" scale="0.001 0.001 0.001"/>
       </geometry>
     </collision>
@@ -97,12 +97,12 @@
       <origin rpy="0 0 ${pi/2}" xyz="0 0 0"/>
       <geometry>
-        <mesh filename="package://interbotix_descriptions/meshes/meshes_vx300/VXA-300-M-3-UA.stl" scale="0.001 0.001 0.001"/>
-      </geometry>
-      <material name="interbotix_black"/>
-    </visual>
-    <collision>
-      <origin rpy="0 0 ${pi/2}" xyz="0 0 0"/>
-      <geometry>
-        <mesh filename="package://interbotix_descriptions/meshes/meshes_vx300/VXA-300-M-3-UA.stl" scale="0.001 0.001 0.001"/>
+        <mesh filename="package://trossen_descriptions/meshes/meshes_vx300/VXA-300-M-3-UA.stl" scale="0.001 0.001 0.001"/>
+      </geometry>
+      <material name="trossen_black"/>
+    </visual>
+    <collision>
+      <origin rpy="0 0 ${pi/2}" xyz="0 0 0"/>
+      <geometry>
+        <mesh filename="package://trossen_descriptions/meshes/meshes_vx300/VXA-300-M-3-UA.stl" scale="0.001 0.001 0.001"/>
       </geometry>
     </collision>
@@ -133,12 +133,12 @@
       <origin rpy="0 0 ${pi/2}" xyz="0 0 0"/>
       <geometry>
-        <mesh filename="package://interbotix_descriptions/meshes/meshes_vx300/VXA-300-M-4-Forearm.stl" scale="0.001 0.001 0.001"/>
-      </geometry>
-      <material name="interbotix_black"/>
-    </visual>
-    <collision>
-      <origin rpy="0 0 ${pi/2}" xyz="0 0 0"/>
-      <geometry>
-        <mesh filename="package://interbotix_descriptions/meshes/meshes_vx300/VXA-300-M-4-Forearm.stl" scale="0.001 0.001 0.001"/>
+        <mesh filename="package://trossen_descriptions/meshes/meshes_vx300/VXA-300-M-4-Forearm.stl" scale="0.001 0.001 0.001"/>
+      </geometry>
+      <material name="trossen_black"/>
+    </visual>
+    <collision>
+      <origin rpy="0 0 ${pi/2}" xyz="0 0 0"/>
+      <geometry>
+        <mesh filename="package://trossen_descriptions/meshes/meshes_vx300/VXA-300-M-4-Forearm.stl" scale="0.001 0.001 0.001"/>
       </geometry>
     </collision>
@@ -169,12 +169,12 @@
       <origin rpy="0 ${pi} ${pi/2}" xyz="0 0 0"/>
       <geometry>
-        <mesh filename="package://interbotix_descriptions/meshes/meshes_vx300/VXA-300-M-5-Wrist.stl" scale="0.001 0.001 0.001"/>
-      </geometry>
-      <material name="interbotix_black"/>
+        <mesh filename="package://trossen_descriptions/meshes/meshes_vx300/VXA-300-M-5-Wrist.stl" scale="0.001 0.001 0.001"/>
+      </geometry>
+      <material name="trossen_black"/>
     </visual>
     <collision>
       <origin rpy="0 ${pi} ${pi/2}" xyz="0 0 0"/>
       <geometry>
-        <mesh filename="package://interbotix_descriptions/meshes/meshes_vx300/VXA-300-M-5-Wrist.stl" scale="0.001 0.001 0.001"/>
+        <mesh filename="package://trossen_descriptions/meshes/meshes_vx300/VXA-300-M-5-Wrist.stl" scale="0.001 0.001 0.001"/>
       </geometry>
     </collision>
@@ -205,12 +205,12 @@
       <origin rpy="0 0 ${pi/2}" xyz="-0.02 0 0"/>
       <geometry>
-        <mesh filename="package://interbotix_descriptions/meshes/meshes_vx300/VXA-300-M-6-Gripper.stl" scale="0.001 0.001 0.001"/>
-      </geometry>
-      <material name="interbotix_black"/>
+        <mesh filename="package://trossen_descriptions/meshes/meshes_vx300/VXA-300-M-6-Gripper.stl" scale="0.001 0.001 0.001"/>
+      </geometry>
+      <material name="trossen_black"/>
     </visual>
     <collision>
       <origin rpy="0 0 ${pi/2}" xyz="-0.02 0 0"/>
       <geometry>
-        <mesh filename="package://interbotix_descriptions/meshes/meshes_vx300/VXA-300-M-6-Gripper.stl" scale="0.001 0.001 0.001"/>
+        <mesh filename="package://trossen_descriptions/meshes/meshes_vx300/VXA-300-M-6-Gripper.stl" scale="0.001 0.001 0.001"/>
       </geometry>
     </collision>
@@ -253,12 +253,12 @@
       <origin rpy="0 0 ${pi/2}" xyz="-0.0685 0 0"/>
       <geometry>
-        <mesh filename="package://interbotix_descriptions/meshes/meshes_vx300/VXA-300-M-7-Gripper-Prop.stl" scale="0.001 0.001 0.001"/>
-      </geometry>
-      <material name="interbotix_black"/>
+        <mesh filename="package://trossen_descriptions/meshes/meshes_vx300/VXA-300-M-7-Gripper-Prop.stl" scale="0.001 0.001 0.001"/>
+      </geometry>
+      <material name="trossen_black"/>
     </visual>
     <collision>
       <origin rpy="0 0 ${pi/2}" xyz="-0.0685 0 0"/>
       <geometry>
-        <mesh filename="package://interbotix_descriptions/meshes/meshes_vx300/VXA-300-M-7-Gripper-Prop.stl" scale="0.001 0.001 0.001"/>
+        <mesh filename="package://trossen_descriptions/meshes/meshes_vx300/VXA-300-M-7-Gripper-Prop.stl" scale="0.001 0.001 0.001"/>
       </geometry>
     </collision>
@@ -281,12 +281,12 @@
         <origin rpy="0 0 ${pi/2}" xyz="-0.063 0 0"/>
         <geometry>
-          <mesh filename="package://interbotix_descriptions/meshes/meshes_vx300/VXA-300-M-8-Gripper-Bar.stl" scale="0.001 0.001 0.001"/>
+          <mesh filename="package://trossen_descriptions/meshes/meshes_vx300/VXA-300-M-8-Gripper-Bar.stl" scale="0.001 0.001 0.001"/>
         </geometry>
-        <material name="interbotix_black"/>
+        <material name="trossen_black"/>
       </visual>
       <collision>
         <origin rpy="0 0 ${pi/2}" xyz="-0.063 0 0"/>
         <geometry>
-          <mesh filename="package://interbotix_descriptions/meshes/meshes_vx300/VXA-300-M-8-Gripper-Bar.stl" scale="0.001 0.001 0.001"/>
+          <mesh filename="package://trossen_descriptions/meshes/meshes_vx300/VXA-300-M-8-Gripper-Bar.stl" scale="0.001 0.001 0.001"/>
         </geometry>
       </collision>
@@ -331,12 +331,12 @@
           <origin rpy="${pi/2} ${-pi} ${pi/2}" xyz="-0.0404 -0.0575 0"/>
           <geometry>
-            <mesh filename="package://interbotix_descriptions/meshes/meshes_vx300/VXA-300-M-9-Finger.stl" scale="0.001 0.001 0.001"/>
+            <mesh filename="package://trossen_descriptions/meshes/meshes_vx300/VXA-300-M-9-Finger.stl" scale="0.001 0.001 0.001"/>
           </geometry>
-          <material name="interbotix_black"/>
+          <material name="trossen_black"/>
         </visual>
         <collision>
           <origin rpy="${pi/2} ${-pi} ${pi/2}" xyz="-0.0404 -0.0575 0"/>
           <geometry>
-            <mesh filename="package://interbotix_descriptions/meshes/meshes_vx300/VXA-300-M-9-Finger.stl" scale="0.001 0.001 0.001"/>
+            <mesh filename="package://trossen_descriptions/meshes/meshes_vx300/VXA-300-M-9-Finger.stl" scale="0.001 0.001 0.001"/>
           </geometry>
         </collision>
@@ -370,12 +370,12 @@
           <origin rpy="${-pi/2} ${pi} ${-pi/2}" xyz="-0.0404 0.0575 0 "/>
           <geometry>
-            <mesh filename="package://interbotix_descriptions/meshes/meshes_vx300/VXA-300-M-9-Finger.stl" scale="0.001 0.001 0.001"/>
+            <mesh filename="package://trossen_descriptions/meshes/meshes_vx300/VXA-300-M-9-Finger.stl" scale="0.001 0.001 0.001"/>
           </geometry>
-          <material name="interbotix_black"/>
+          <material name="trossen_black"/>
         </visual>
         <collision>
           <origin rpy="${-pi/2} ${pi} ${-pi/2}" xyz="-0.0404 0.0575 0 "/>
           <geometry>
-            <mesh filename="package://interbotix_descriptions/meshes/meshes_vx300/VXA-300-M-9-Finger.stl" scale="0.001 0.001 0.001"/>
+            <mesh filename="package://trossen_descriptions/meshes/meshes_vx300/VXA-300-M-9-Finger.stl" scale="0.001 0.001 0.001"/>
           </geometry>
         </collision>
