Commit message: feat: refactor URDF loading, add Jaco model, fix collision and deepcopy
URDFRobot / model loading:
- Introduce URDFRobot.py with URDF_file() and URDF_read() module-level
  functions; all URDF models converted to explicit super().__init__(urdf_path,
  manufacturer) args (Group 2: UR*, Trossen, Puma560, LBR, AL5D, KinovaGen3)
- Robot.URDF() classmethod formally deprecated with migration message
- _load_urdf_from_RD() now supports both URDF_PATH and XACRO_PATH from
  robot_descriptions (comment explains the per-model variation)
- _parse_urdf() raises RuntimeError if a link has <collision> elements but
  none load, catching silent mesh resolution failures early
- qut_frankie_description xacro files: replace franka_description package
  references throughout; Panda restored to ship with local xacro
- PR2 hardcoded joint count (31) replaced with self.n

Mico → Jaco:
- Remove broken URDF Mico model (kinova_description not in rtbdata)
- Add Jaco model (j2n6s200, 6-DOF) loaded from robot_descriptions
- DH/Mico model unchanged

models.list():
- Catch all exceptions when instantiating models, not just TypeError;
  add missing continue so a failed load doesn't NameError on robot.structure

Link deepcopy:
- Add _copy_shapes() helper that skips coal CollisionObject instances
  (which don't support pickling) and warns once per link if shapes are lost
- Use in both Link.__deepcopy__ and DHLink.__deepcopy__

Add tech-debt.md documenting the root-cause shared-state issue (Option 2)

File: rtb-data/rtbdata/xacro/qut_frankie_description/robots/dual_panda_example.urdf.xacro (robot description, xacro)
@@ -3,6 +3,6 @@
   <xacro:arg name="arm_id_1" default="panda_1" />
   <xacro:arg name="arm_id_2" default="panda_2" />
-  <xacro:include filename="$(find franka_description)/robots/panda_arm.xacro"/>
-  <xacro:include filename="$(find franka_description)/robots/hand.xacro"/>
+  <xacro:include filename="$(find qut_frankie_description)/robots/panda_arm.xacro"/>
+  <xacro:include filename="$(find qut_frankie_description)/robots/hand.xacro"/>
   <!-- box shaped table as base for the 2 Pandas -->
   <link name="base">

File: rtb-data/rtbdata/xacro/qut_frankie_description/robots/frankieOmni_arm.urdf.xacro (robot description, xacro)
@@ -1,5 +1,5 @@
 <?xml version='1.0' encoding='utf-8'?>
 <robot xmlns:xacro="http://www.ros.org/wiki/xacro" name="frankie">
-  <xacro:include filename="$(find franka_description)/robots/frankieOmni_arm.xacro" />
+  <xacro:include filename="$(find qut_frankie_description)/robots/frankieOmni_arm.xacro" />
   <xacro:panda_arm safety_distance="0.00"/>
 </robot>

File: rtb-data/rtbdata/xacro/qut_frankie_description/robots/frankieOmni_arm.xacro (robot description, xacro)
@@ -3,5 +3,5 @@
   <!-- safety_distance: Minimum safety distance in [m] by which the collision volumes are expanded and which is enforced during robot motions -->
   <!-- arm_id: Namespace of the panda arm. Serves to differentiate between arms in case of multiple instances. -->
-  <xacro:macro name="panda_arm" params="arm_id:='panda' description_pkg:='franka_description' connected_to:='' xyz:='0 0 0' rpy:='0 0 0' safety_distance:=0">
+  <xacro:macro name="panda_arm" params="arm_id:='panda' description_pkg:='qut_frankie_description' connected_to:='' xyz:='0 0 0' rpy:='0 0 0' safety_distance:=0">
     <xacro:unless value="${not connected_to}">
       <joint name="${arm_id}_joint_${connected_to}" type="fixed">

File: rtb-data/rtbdata/xacro/qut_frankie_description/robots/frankieOmni_arm_hand.urdf.xacro (robot description, xacro)
@@ -1,6 +1,6 @@
 <?xml version="1.0" encoding="utf-8"?>
 <robot xmlns:xacro="http://www.ros.org/wiki/xacro" name="frankie">
-  <xacro:include filename="$(find franka_description)/robots/frankieOmni_arm.xacro"/>
-  <xacro:include filename="$(find franka_description)/robots/hand.xacro"/>
+  <xacro:include filename="$(find qut_frankie_description)/robots/frankieOmni_arm.xacro"/>
+  <xacro:include filename="$(find qut_frankie_description)/robots/hand.xacro"/>
   <xacro:panda_arm safety_distance="0.00"/>
   <xacro:hand ns="frankie" rpy="0 0 ${-pi/4}" connected_to="panda_link8" safety_distance="0.00"/>

File: rtb-data/rtbdata/xacro/qut_frankie_description/robots/frankie_arm.urdf.xacro (robot description, xacro)
@@ -1,5 +1,5 @@
 <?xml version='1.0' encoding='utf-8'?>
 <robot xmlns:xacro="http://www.ros.org/wiki/xacro" name="frankie">
-  <xacro:include filename="$(find franka_description)/robots/frankie_arm.xacro" />
+  <xacro:include filename="$(find qut_frankie_description)/robots/frankie_arm.xacro" />
   <xacro:panda_arm safety_distance="0.00"/>
 </robot>

File: rtb-data/rtbdata/xacro/qut_frankie_description/robots/frankie_arm.xacro (robot description, xacro)
@@ -3,5 +3,5 @@
   <!-- safety_distance: Minimum safety distance in [m] by which the collision volumes are expanded and which is enforced during robot motions -->
   <!-- arm_id: Namespace of the panda arm. Serves to differentiate between arms in case of multiple instances. -->
-  <xacro:macro name="panda_arm" params="arm_id:='panda' description_pkg:='franka_description' connected_to:='' xyz:='0 0 0' rpy:='0 0 0' safety_distance:=0">
+  <xacro:macro name="panda_arm" params="arm_id:='panda' description_pkg:='qut_frankie_description' connected_to:='' xyz:='0 0 0' rpy:='0 0 0' safety_distance:=0">
     <xacro:unless value="${not connected_to}">
       <joint name="${arm_id}_joint_${connected_to}" type="fixed">

File: rtb-data/rtbdata/xacro/qut_frankie_description/robots/frankie_arm_hand.urdf.xacro (robot description, xacro)
@@ -1,6 +1,6 @@
 <?xml version="1.0" encoding="utf-8"?>
 <robot xmlns:xacro="http://www.ros.org/wiki/xacro" name="frankie">
-  <xacro:include filename="$(find franka_description)/robots/frankie_arm.xacro"/>
-  <xacro:include filename="$(find franka_description)/robots/hand.xacro"/>
+  <xacro:include filename="$(find qut_frankie_description)/robots/frankie_arm.xacro"/>
+  <xacro:include filename="$(find qut_frankie_description)/robots/hand.xacro"/>
   <xacro:panda_arm safety_distance="0.00"/>
   <xacro:hand ns="frankie" rpy="0 0 ${-pi/4}" connected_to="panda_link8" safety_distance="0.00"/>

File: rtb-data/rtbdata/xacro/qut_frankie_description/robots/hand.xacro (robot description, xacro)
@@ -13,5 +13,5 @@
       <visual>
         <geometry>
-          <mesh filename="package://franka_description/meshes/visual/hand.dae"/>
+          <mesh filename="package://qut_frankie_description/meshes/visual/hand.dae"/>
         </geometry>
       </visual>
@@ -56,5 +56,5 @@
       <visual>
         <geometry>
-          <mesh filename="package://franka_description/meshes/visual/finger.dae"/>
+          <mesh filename="package://qut_frankie_description/meshes/visual/finger.dae"/>
         </geometry>
       </visual>
@@ -64,5 +64,5 @@
         <origin xyz="0 0 0" rpy="0 0 ${pi}"/>
         <geometry>
-          <mesh filename="package://franka_description/meshes/visual/finger.dae"/>
+          <mesh filename="package://qut_frankie_description/meshes/visual/finger.dae"/>
         </geometry>
       </visual>

File: rtb-data/rtbdata/xacro/qut_frankie_description/robots/panda_arm.urdf.xacro (robot description, xacro)
@@ -1,5 +1,5 @@
 <?xml version='1.0' encoding='utf-8'?>
 <robot xmlns:xacro="http://www.ros.org/wiki/xacro" name="panda">
-  <xacro:include filename="$(find franka_description)/robots/panda_arm.xacro" />
+  <xacro:include filename="$(find qut_frankie_description)/robots/panda_arm.xacro" />
   <xacro:panda_arm safety_distance="0.00"/>
 </robot>

File: rtb-data/rtbdata/xacro/qut_frankie_description/robots/panda_arm.xacro (robot description, xacro)
@@ -3,5 +3,5 @@
   <!-- safety_distance: Minimum safety distance in [m] by which the collision volumes are expanded and which is enforced during robot motions -->
   <!-- arm_id: Namespace of the panda arm. Serves to differentiate between arms in case of multiple instances. -->
-  <xacro:macro name="panda_arm" params="arm_id:='panda' description_pkg:='franka_description' connected_to:='' xyz:='0 0 0' rpy:='0 0 0' safety_distance:=0">
+  <xacro:macro name="panda_arm" params="arm_id:='panda' description_pkg:='qut_frankie_description' connected_to:='' xyz:='0 0 0' rpy:='0 0 0' safety_distance:=0">
     <xacro:unless value="${not connected_to}">
       <joint name="${arm_id}_joint_${connected_to}" type="fixed">

File: rtb-data/rtbdata/xacro/qut_frankie_description/robots/panda_arm_hand.urdf.xacro (robot description, xacro)
@@ -1,6 +1,6 @@
 <?xml version="1.0" encoding="utf-8"?>
 <robot xmlns:xacro="http://www.ros.org/wiki/xacro" name="panda">
-  <xacro:include filename="$(find franka_description)/robots/panda_arm.xacro"/>
-  <xacro:include filename="$(find franka_description)/robots/hand.xacro"/>
+  <xacro:include filename="$(find qut_frankie_description)/robots/panda_arm.xacro"/>
+  <xacro:include filename="$(find qut_frankie_description)/robots/hand.xacro"/>
   <xacro:panda_arm safety_distance="0.00"/>
   <xacro:hand ns="panda" rpy="0 0 ${-pi/4}" connected_to="panda_link8" safety_distance="0.00"/>
